File: reference/CM4IO-KiCAD/USB2-HUB.kicad_sch (KiCad schematic)
At the start: 32 parts, among them J11 USB_OTG, J13 690-008-221-904, J14 Conn_02x05_Odd_Even, U13 FSUSB42MUX, U4 TPD4EUSB30, U6 USB2514B-I/M2, U7 AP22653W6, Y1 24MHz

Commit message: Schaltplan Update
Other:
- moved on the sheet: J13
