File: reference/CM4IO-KiCAD/PSUs.kicad_sch (KiCad schematic)
At the start: 33 parts, among them J19 Barrel_Jack, J20 AMP171826-4, Q1 DMP3013SFV-7, U16 AP64501SP-13

Commit message: Save.
Changed lines of the file:
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@@
   )
   (text "Ideal diode to prevent reverse\npolarity at the input"
-    (at 96.52 36.83 0)
+    (at 95.25 36.83 0)
     (effects (font (size 1.27 1.27)) (justify left bottom))
   )
