File: reference/ttude-rpi-3b-carrier/KiCad/main_backupboard_1.kicad_sch (KiCad schematic)
At the start: 38 parts, among them IC1 D36V28FX, IC2 D36V28FX, U1 RASPBERRY_PI_3_MODEL_B+, X1 MICROMATCH-4, X2 MICROMATCH-10, X3 MICROMATCH-4, X5 MICROMATCH-10

Commit message: Save.
Other:
- moved on the sheet: JP1, JP4
Changed lines of the file:
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@@
   (junction (at 353.695 80.645) (diameter 0) (color 0 0 0 0)
   )
+  (junction (at 39.37 247.65) (diameter 0) (color 0 0 0 0)
+  )
   (junction (at 205.105 321.945) (diameter 0) (color 0 0 0 0)
   )
@@
   (junction (at 359.41 158.115) (diameter 0) (color 0 0 0 0)
   )
-  (junction (at 39.37 254.635) (diameter 0) (color 0 0 0 0)
-  )
   (junction (at 114.935 165.1) (diameter 0) (color 0 0 0 0)
   )
@@
   (junction (at 393.065 167.64) (diameter 0) (color 0 0 0 0)
   )
-  (junction (at 52.07 254.635) (diameter 0) (color 0 0 0 0)
-  )
   (junction (at 415.925 167.64) (diameter 0) (color 0 0 0 0)
   )
@@
   (junction (at 210.185 263.525) (diameter 0) (color 0 0 0 0)
   )
+  (junction (at 39.37 271.78) (diameter 0) (color 0 0 0 0)
+  )
   (junction (at 415.925 152.4) (diameter 0) (color 0 0 0 0)
   )
@@
   (junction (at 39.37 239.395) (diameter 0) (color 0 0 0 0)
   )
-  (junction (at 39.37 247.015) (diameter 0) (color 0 0 0 0)
-  )
   (junction (at 107.315 175.26) (diameter 0) (color 0 0 0 0)
   )
@@
   (junction (at 72.39 236.855) (diameter 0) (color 0 0 0 0)
   )
+  (junction (at 54.61 254.635) (diameter 0) (color 0 0 0 0)
+  )
   (junction (at 114.935 162.56) (diameter 0) (color 0 0 0 0)
   )
@@
   (junction (at 39.37 262.255) (diameter 0) (color 0 0 0 0)
   )
-  (wire (pts (xy 46.99 247.015) (xy 39.37 247.015))
+  (wire (pts (xy 49.53 247.65) (xy 39.37 247.65))
     (stroke (width 0.1524) (type solid))
   )
@@
     (stroke (width 0.1524) (type solid))
   )
+  (wire (pts (xy 60.96 271.78) (xy 60.96 257.81))
+    (stroke (width 0) (type default))
+  )
   (wire (pts (xy 438.785 167.64) (xy 438.785 162.56))
     (stroke (width 0.1524) (type solid))
@@
     (stroke (width 0.1524) (type solid))
   )
+  (wire (pts (xy 39.37 271.78) (xy 39.37 262.255))
+    (stroke (width 0.1524) (type solid))
+  )
   (wire (pts (xy 132.715 165.1) (xy 125.095 165.1))
     (stroke (width 0.1524) (type solid))
@@
     (stroke (width 0.1524) (type solid))
   )
+  (wire (pts (xy 60.96 257.81) (xy 52.07 257.81))
+    (stroke (width 0) (type default))
+  )
   (wire (pts (xy 142.875 175.26) (xy 135.255 175.26))
     (stroke (width 0.1524) (type solid))
   )
-  (wire (pts (xy 39.37 262.255) (xy 39.37 254.635))
-    (stroke (width 0.1524) (type solid))
-  )
-  (wire (pts (xy 39.37 272.415) (xy 39.37 262.255))
+  (wire (pts (xy 39.37 272.415) (xy 39.37 271.78))
     (stroke (width 0.1524) (type solid))
   )
@@
     (stroke (width 0.1524) (type solid))
   )
-  (wire (pts (xy 44.45 254.635) (xy 39.37 254.635))
+  (wire (pts (xy 53.34 271.78) (xy 39.37 271.78))
     (stroke (width 0.1524) (type solid))
   )
@@
     (stroke (width 0.1524) (type solid))
   )
+  (wire (pts (xy 54.61 254.635) (xy 52.07 254.635))
+    (stroke (width 0.1524) (type solid))
+  )
   (wire (pts (xy 398.145 238.125) (xy 398.145 240.665))
     (stroke (width 0.1524) (type solid))
   )
+  (wire (pts (xy 54.61 254.635) (xy 72.39 254.635))
+    (stroke (width 0.1524) (type solid))
+  )
   (wire (pts (xy 197.485 309.245) (xy 197.485 304.165))
     (stroke (width 0.1524) (type solid))
@@
     (stroke (width 0.1524) (type solid))
   )
-  (wire (pts (xy 52.07 247.015) (xy 52.07 254.635))
-    (stroke (width 0.1524) (type solid))
+  (wire (pts (xy 54.61 247.65) (xy 54.61 254.635))
+    (stroke (width 0.1524) (type solid))
+  )
+  (wire (pts (xy 52.07 257.81) (xy 52.07 254.635))
+    (stroke (width 0) (type default))
   )
   (wire (pts (xy 72.39 236.855) (xy 77.47 236.855))
@@
     (stroke (width 0.1524) (type solid))
   )
+  (wire (pts (xy 39.37 247.65) (xy 39.37 262.255))
+    (stroke (width 0.1524) (type solid))
+  )
   (wire (pts (xy 127.635 180.34) (xy 117.475 180.34))
     (stroke (width 0.1524) (type solid))
@@
     (stroke (width 0.1524) (type solid))
   )
-  (wire (pts (xy 39.37 254.635) (xy 39.37 247.015))
-    (stroke (width 0.1524) (type solid))
-  )
   (wire (pts (xy 114.935 165.1) (xy 107.315 172.72))
     (stroke (width 0.1524) (type solid))
@@
     (stroke (width 0.1524) (type solid))
   )
-  (wire (pts (xy 52.07 254.635) (xy 72.39 254.635))
-    (stroke (width 0.1524) (type solid))
-  )
   (wire (pts (xy 295.275 42.545) (xy 291.465 42.545))
     (stroke (width 0.1524) (type solid))
@@
     (stroke (width 0.1524) (type solid))
   )
-  (wire (pts (xy 39.37 247.015) (xy 39.37 239.395))
+  (wire (pts (xy 39.37 239.395) (xy 39.37 247.65))
     (stroke (width 0.1524) (type solid))
   )
@@
   (wire (pts (xy 537.845 148.59) (xy 537.845 140.97))
     (stroke (width 0.1524) (type solid))
+  )
+  (rectangle (start 283.21 12.7) (end 383.54 96.52)
+    (stroke (width 0) (type default))
+    (fill (type none))
+  )
+  (rectangle (start 328.93 208.28) (end 447.04 251.46)
+    (stroke (width 0) (type default))
+    (fill (type none))
+  )
+  (rectangle (start 123.19 241.3) (end 264.16 335.28)
+    (stroke (width 0) (type default))
+    (fill (type none))
+  )
+  (rectangle (start 46.99 162.56) (end 99.06 210.82)
+    (stroke (width 0) (type default))
+    (fill (type none))
+  )
+  (rectangle (start 473.71 133.35) (end 546.1 179.07)
+    (stroke (width 0) (type default))
+    (fill (type none))
   )
   (label "DATA" (at 530.225 166.37 0) (fields_autoplaced)
@@
     )
   )
-  (symbol (lib_id "main_backupboard-eagle-import:PINHD-1X3") (at 49.53 249.555 270) (unit 1)
-    (in_bom yes) (on_board yes) (dnp no)
-    (property "Reference" "JP1" (at 55.245 243.205 0)
-      (effects (font (size 1.778 1.5113)) (justify left bottom))
-    )
-    (property "Value" "8V-Buchse" (at 41.91 243.205 0)
-      (effects (font (size 1.778 1.5113)) (justify left bottom))
-    )
-    (property "Footprint" "main_backupboard:1X03" (at 49.53 249.555 0)
-      (effects (font (size 1.27 1.27)) hide)
-    )
-    (property "Datasheet" "" (at 49.53 249.555 0)
+  (symbol (lib_id "main_backupboard-eagle-import:PINHD-1X3") (at 52.07 250.19 270) (unit 1)
+    (in_bom yes) (on_board yes) (dnp no)
+    (property "Reference" "JP1" (at 57.785 243.84 0)
+      (effects (font (size 1.778 1.5113)) (justify left bottom))
+    )
+    (property "Value" "8V-Buchse" (at 44.45 243.84 0)
+      (effects (font (size 1.778 1.5113)) (justify left bottom))
+    )
+    (property "Footprint" "main_backupboard:1X03" (at 52.07 250.19 0)
+      (effects (font (size 1.27 1.27)) hide)
+    )
+    (property "Datasheet" "" (at 52.07 250.19 0)
       (effects (font (size 1.27 1.27)) hide)
     )
@@
     )
   )
-  (symbol (lib_id "main_backupboard-eagle-import:PINHD-1X4") (at 46.99 257.175 270) (unit 1)
-    (in_bom yes) (on_board yes) (dnp no)
-    (property "Reference" "JP4" (at 55.245 250.825 0)
-      (effects (font (size 1.778 1.5113)) (justify left bottom))
-    )
-    (property "Value" "12V-Buchse" (at 39.37 250.825 0)
-      (effects (font (size 1.778 1.5113)) (justify left bottom))
-    )
-    (property "Footprint" "main_backupboard:1X04" (at 46.99 257.175 0)
-      (effects (font (size 1.27 1.27)) hide)
-    )
-    (property "Datasheet" "" (at 46.99 257.175 0)
-      (effects (font (size 1.27 1.27)) hide)
-    )
+  (symbol (lib_id "main_backupboard-eagle-import:PINHD-1X4") (at 55.88 274.32 270) (unit 1)
+    (in_bom yes) (on_board yes) (dnp no)
+    (property "Reference" "JP4" (at 64.135 267.97 0)
+      (effects (font (size 1.778 1.5113)) (justify left bottom))
+    )
+    (property "Value" "12V-Buchse" (at 48.26 267.97 0)
+      (effects (font (size 1.778 1.5113)) (justify left bottom))
+    )
+    (property "Footprint" "main_backupboard:1X04" (at 55.88 274.32 0)
+      (effects (font (size 1.27 1.27)) hide)
+    )
+    (property "Datasheet" "" (at 55.88 274.32 0)
+      (effects (font (size 1.27 1.27)) hide)
+    )
